Commit message: Changes for demo

File: attachable_pkg/models/other/myfirst.xacro (robot description, xacro)
@@ -17,3 +17,3 @@
   <xacro:body sufix="1">
   </xacro:body>
-  <xacro:leg sufix="1"/><joint name="AttachableJoint_1body1_1leg1" type="fixed"><parent link="AttachableLink_1_body_1"/><child link="AttachableLink_1_leg_1"/><origin rpy="0 0 0" xyz="0 0 0"/></joint></robot>
+  <xacro:leg sufix="1"/><joint name="AttachableJoint_1body1_1leg1" type="fixed"><parent link="AttachableLink_1_body_1"/><child link="AttachableLink_1_leg_1"/><origin rpy="0 0 0" xyz="0 0 0"/></joint><xacro:leg sufix="1"/><joint name="AttachableJoint_1body1_1leg1" type="fixed"><parent link="AttachableLink_1_body_1"/><child link="AttachableLink_1_leg_1"/><origin rpy="0 0 0" xyz="0 0 0"/></joint></robot>

Commit message: Update launchfiles

File: attachable_pkg/models/other/myfirst.xacro (robot description, xacro)
@@ -17,3 +17,3 @@
   <xacro:body sufix="1">
   </xacro:body>
-  <xacro:leg sufix="1"/><joint name="AttachableJoint_1body1_1leg1" type="fixed"><parent link="AttachableLink_1_body_1"/><child link="AttachableLink_1_leg_1"/><origin rpy="0 0 0" xyz="0 0 0"/></joint><xacro:leg sufix="1"/><joint name="AttachableJoint_1body1_1leg1" type="fixed"><parent link="AttachableLink_1_body_1"/><child link="AttachableLink_1_leg_1"/><origin rpy="0 0 0" xyz="0 0 0"/></joint></robot>
+  </robot>

File: attachable_pkg/models/xacro_files/import_path.xacro (robot description, xacro)
@@ -1,5 +1,7 @@
 <?xml version="1.0"?>
 <robot name="imports" xmlns:xacro="http://wiki.ros.org/xacro">
-  <xacro:include filename="../models/rm2_body.xacro" />
-  <xacro:include filename="../models/rm2_leg.xacro" />
+  <!--xacro:include filename="../models/rm2_body.xacro" />
+  <xacro:include filename="../models/rm2_leg.xacro" /-->
+  <xacro:include filename="$(find attachable_pkg)/models/xacro_files/rm2_body.xacro"/>
+  <xacro:include filename="$(find attachable_pkg)/models/xacro_files/rm2_leg.xacro" />
 </robot>
